File: Hardware/ETH2CDSO1B/ETH2CDSO1B.kicad_sch (KiCad schematic)
At the start: 0 parts

Commit message: Hardware
Other:
- added sheet ADC (ADC.kicad_sch)
- added sheet CH2 Input (CH2_Input.kicad_sch)
- added sheet FPGA (FPGA.kicad_sch)
- added sheet Power (Power.kicad_sch)
- sheet CH1 Input ports: added REF_OUT_AD9288_CH1; removed none
- sheet Voltage Source ports: added DAC_~{CLR}, DAC_~{LDAC}, OFFSET1_CH1, OFFSET1_CH2, OFFSET2_CH1, OFFSET2_CH2, OFFSET3_CH1, OFFSET3_CH2, SELFCAL, SELF_CAL_CH1, SELF_CAL_CH2, SPI_CS3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; removed none
