File: Hardware/ETH2CDSO1B/CH1_Input.kicad_sch (KiCad schematic)
At the start: 90 parts, among them J201 73251-1153, K201 G6K-2F-Y-DC5, K202 G6K-2F-Y-DC5, Q201 MMBFJ309LT1G, Q202 BC846B, Q203 MMBTH10LT3G, Q204 BC846B, U201 AQY280S, U202 AD8510ARZ, U203 AD8370AREZ, U204 SN74HC595PWRG4, U205 LMH6552MA

Commit message: Hardware
Parts:
- added J202: RFShield_OnePiece, symbol Device:RFShield_OnePiece
- added TP201, TP202, TP203, TP204, TP205: TP, TestPoint:TestPoint_Pad_2.0x2.0mm, symbol Connector:TestPoint
Connections:
- net GND: now also J202.1 (Shield)
- net OFFSET2_CH1: now also TP205.1
- net at C212.2, R216.1, U201.3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: now also TP203.1
- net at Q203.2 (E), R222.2, R227.1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: now also TP204.1
- net at C214.1, K202.3, R214.1: now also TP202.1
- net REF_OUT_AD9288_CH1: now reaches C233.1, U205.2 (VCM)
- net at J201.1 (In), R201.1, R204.2: now also TP201.1
Other:
- moved on the sheet: R235, R236, RN201, RN202, U205

Commit message: Hardware
Connections:
- net +12V: no longer C215.2, D201.1 (K), FB203.1
- net +5V: now also C215.2, D201.1 (K), FB203.1
Changed lines of the file:
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@@
     )
   )
-  (symbol (lib_id "Device:R") (at 178.435 200.66 90) (unit 1)
+  (symbol (lib_id "power:+5V") (at 189.23 82.55 0) (unit 1)
     (in_bom yes) (on_board yes) (dnp no) (fields_autoplaced)
-    (property "Reference" "R222" (at 178.435 194.945 90)
-      (effects (font (size 1.27 1.27)))
+    (property "Reference" "#PWR0233" (at 189.23 86.36 0)
+      (effects (font (size 1.27 1.27)) hide)
     )
-    (property "Value" "806k" (at 178.435 197.485 90)
+    (property "Value" "+5V" (at 189.23 78.105 0)
       (effects (font (size 1.27 1.27)))
     )
-    (property "Footprint" "Resistor_SMD:R_0603_1608Metric_Pad0.98x0.95mm_HandSolder" (at 178.435 202.438 90)
+    (property "Footprint" "" (at 189.23 82.55 0)
       (effects (font (size 1.27 1.27)) hide)
     )
-    (property "Datasheet" "~" (at 178.435 200.66 0)
+    (property "Datasheet" "" (at 189.23 82.55 0)
       (effects (font (size 1.27 1.27)) hide)
     )
     (pin "1")
-    (pin "2")
     (instances
       (project "ETH2CDSO1B"
         (path "/5e9d9a67-9011-4d17-9f7a-23dbb04d2fbf/4548d26a-48b5-4733-ae40-ebee8ab230ff"
-          (reference "R222") (unit 1)
+          (reference "#PWR0233") (unit 1)
         )
       )
     )
   )
-  (symbol (lib_id "power:+12V") (at 189.23 82.55 0) (unit 1)
+  (symbol (lib_id "Device:R") (at 178.435 200.66 90) (unit 1)
     (in_bom yes) (on_board yes) (dnp no) (fields_autoplaced)
-    (property "Reference" "#PWR0233" (at 189.23 86.36 0)
-      (effects (font (size 1.27 1.27)) hide)
+    (property "Reference" "R222" (at 178.435 194.945 90)
+      (effects (font (size 1.27 1.27)))
     )
-    (property "Value" "+12V" (at 189.23 78.105 0)
+    (property "Value" "806k" (at 178.435 197.485 90)
       (effects (font (size 1.27 1.27)))
     )
-    (property "Footprint" "" (at 189.23 82.55 0)
+    (property "Footprint" "Resistor_SMD:R_0603_1608Metric_Pad0.98x0.95mm_HandSolder" (at 178.435 202.438 90)
       (effects (font (size 1.27 1.27)) hide)
     )
-    (property "Datasheet" "" (at 189.23 82.55 0)
+    (property "Datasheet" "~" (at 178.435 200.66 0)
       (effects (font (size 1.27 1.27)) hide)
     )
     (pin "1")
+    (pin "2")
     (instances
       (project "ETH2CDSO1B"
         (path "/5e9d9a67-9011-4d17-9f7a-23dbb04d2fbf/4548d26a-48b5-4733-ae40-ebee8ab230ff"
-          (reference "#PWR0233") (unit 1)
+          (reference "R222") (unit 1)
         )
       )
@@
     )
   )
+  (symbol (lib_id "power:+5V") (at 144.78 109.22 90) (unit 1)
+    (in_bom yes) (on_board yes) (dnp no) (fields_autoplaced)
+    (property "Reference" "#PWR0226" (at 148.59 109.22 0)
+      (effects (font (size 1.27 1.27)) hide)
+    )
+    (property "Value" "+5V" (at 141.605 109.22 90)
+      (effects (font (size 1.27 1.27)) (justify left))
+    )
+    (property "Footprint" "" (at 144.78 109.22 0)
+      (effects (font (size 1.27 1.27)) hide)
+    )
+    (property "Datasheet" "" (at 144.78 109.22 0)
+      (effects (font (size 1.27 1.27)) hide)
+    )
+    (pin "1")
+    (instances
+      (project "ETH2CDSO1B"
+        (path "/5e9d9a67-9011-4d17-9f7a-23dbb04d2fbf/4548d26a-48b5-4733-ae40-ebee8ab230ff"
+          (reference "#PWR0226") (unit 1)
+        )
+      )
+    )
+  )
   (symbol (lib_id "Device:R") (at 95.885 178.435 0) (unit 1)
     (in_bom yes) (on_board yes) (dnp no)
@@
         )
       )
-    )
-  )
-  (symbol (lib_id "power:+12V") (at 144.78 109.22 90) (unit 1)
-    (in_bom yes) (on_board yes) (dnp no) (fields_autoplaced)
-    (property "Reference" "#PWR0226" (at 148.59 109.22 0)
-      (effects (font (size 1.27 1.27)) hide)
-    )
-    (property "Value" "+12V" (at 140.97 109.22 90)
-      (effects (font (size 1.27 1.27)) (justify left))
-    )
-    (property "Footprint" "" (at 144.78 109.22 0)
-      (effects (font (size 1.27 1.27)) hide)
-    )
-    (property "Datasheet" "" (at 144.78 109.22 0)
-      (effects (font (size 1.27 1.27)) hide)
-    )
-    (pin "1")
-    (instances
-      (project "ETH2CDSO1B"
-        (path "/5e9d9a67-9011-4d17-9f7a-23dbb04d2fbf/4548d26a-48b5-4733-ae40-ebee8ab230ff"
-          (reference "#PWR0226") (unit 1)
-        )
-      )

Commit message: Hardware
Parts:
- removed C204: 2p2, Capacitor_SMD:C_0603_1608Metric_Pad1.08x0.95mm_HandSolder, symbol Device:C
- removed C210: 100p, Capacitor_SMD:C_0603_1608Metric_Pad1.08x0.95mm_HandSolder, symbol Device:C
- removed R210: 10, Resistor_SMD:R_0603_1608Metric_Pad0.98x0.95mm_HandSolder, symbol Device:R
- removed R211: 12, Resistor_SMD:R_0603_1608Metric_Pad0.98x0.95mm_HandSolder, symbol Device:R
- added C206: 11p, Capacitor_SMD:C_0603_1608Metric_Pad1.08x0.95mm_HandSolder, symbol Device:C
- added R202: 17R8, Resistor_SMD:R_0603_1608Metric_Pad0.98x0.95mm_HandSolder, symbol Device:R
- added R205: 150, Resistor_SMD:R_0603_1608Metric_Pad0.98x0.95mm_HandSolder, symbol Device:R
- added R208: 24k9, Resistor_SMD:R_1206_3216Metric_Pad1.30x1.75mm_HandSolder, symbol Device:R
- added R213: 100, Resistor_SMD:R_0603_1608Metric_Pad0.98x0.95mm_HandSolder, symbol Device:R
- C204: renamed from C207; value 2p2 -> 22p
- C208: renamed from C205; value 12p -> 27p
- R204: value 33R2 -> 4R7
- R207: value 38k3 -> 22k6
- R209: renamed from R205; value 976k -> 953k
- R228: renamed from R226; value 100 -> 249
- R230: renamed from R228; value 100 -> 75
- renumbered C208 to C203, C203 to C205, C206 to C207, C211 to C210, C212 to C211, C213 to C212, C214 to C213, C215 to C214, C216 to C215, C217 to C216, C218 to C217, C219 to C218, C220 to C219, C221 to C220, C222 to C221, C223 to C222, C224 to C223, C225 to C224, C226 to C225, C227 to C226, C228 to C227, C229 to C228, C230 to C229, C231 to C230, C232 to C231, C233 to C232, R208 to R210, R209 to R211, R202 to R212, R212 to R214, R213 to R215, R214 to R216, R215 to R217, R216 to R218, R217 to R219, R218 to R220, R219 to R221, R220 to R222, R221 to R223, R222 to R224, R223 to R225, R224 to R226, R225 to R227, R227 to R229, R229 to R231, R230 to R232, R231 to R233, R232 to R234, R233 to R235, R234 to R236, R235 to R237, R236 to R238
Connections:
- net +12V: no longer U202.7 (V+)
- net +5V: now also U202.7 (V+)
- net GND: now also C203.2, C204.2, C206.2
- net at K202.4: now also R213.2
- net at K202.5, R209.1: now also C208.1, R205.2; no longer R212.2
- net at C203.1, C204.1: now also R202.1; no longer C208.2
- net at R212.1: now also R207.1, R202.2, R208.2, R213.1; no longer C208.1
- net +5FC1 renamed +5FC2
- net -5FC1 renamed -5FC2
- new net: C208.2, R212.2
- new net: C206.1, R205.1
- new net: R208.1, R209.2
Other:
- moved on the sheet: C203, C204, C205, C207, C208, C222, C223, FB202, R207, R209, R212, R231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
