File: Hardware/ETH2CDSO1B/CH2_Input.kicad_sch (KiCad schematic)
At the start: 96 parts, among them J201 73251-1153, J202 RFShield_OnePiece, K201 G6K-2F-Y-DC5, K202 G6K-2F-Y-DC5, Q201 MMBFJ309LT1G, Q202 BC846B, Q203 MMBTH10LT3G, Q204 BC846B, U201 AQY280S, U202 AD8510ARZ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

Commit message: Hardware
Connections:
- net +12V: no longer C215.2, D201.1 (K), FB203.1
- net +5V: now also C215.2, D201.1 (K), FB203.1
Changed lines of the file:
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@@
-    )
-  )
-  (symbol (lib_id "power:+12V") (at 141.605 110.49 90) (unit 1)
-    (in_bom yes) (on_board yes) (dnp no) (fields_autoplaced)
-    (property "Reference" "#PWR0226" (at 145.415 110.49 0)
-      (effects (font (size 1.27 1.27)) hide)
-    )
-    (property "Value" "+12V" (at 137.795 110.49 90)
-      (effects (font (size 1.27 1.27)) (justify left))
-    )
-    (property "Footprint" "" (at 141.605 110.49 0)
-      (effects (font (size 1.27 1.27)) hide)
-    )
-    (property "Datasheet" "" (at 141.605 110.49 0)
-      (effects (font (size 1.27 1.27)) hide)
-    )
-    (pin "1")
-    (instances
-      (project "ETH2CDSO1B"
-        (path "/5e9d9a67-9011-4d17-9f7a-23dbb04d2fbf/4548d26a-48b5-4733-ae40-ebee8ab230ff"
-          (reference "#PWR0226") (unit 1)
-        )
-        (path "/5e9d9a67-9011-4d17-9f7a-23dbb04d2fbf/45cf2216-7ba0-412c-bbcb-6adbd9bfb27f"
-          (reference "#PWR0426") (unit 1)
-        )
-      )
     )
   )
@@
         (path "/5e9d9a67-9011-4d17-9f7a-23dbb04d2fbf/45cf2216-7ba0-412c-bbcb-6adbd9bfb27f"
           (reference "R414") (unit 1)
+        )
+      )
+    )
+  )
+  (symbol (lib_id "power:+5V") (at 141.605 110.49 90) (unit 1)
+    (in_bom yes) (on_board yes) (dnp no) (fields_autoplaced)
+    (property "Reference" "#PWR0215" (at 145.415 110.49 0)
+      (effects (font (size 1.27 1.27)) hide)
+    )
+    (property "Value" "+5V" (at 137.795 110.49 90)
+      (effects (font (size 1.27 1.27)) (justify left))
+    )
+    (property "Footprint" "" (at 141.605 110.49 0)
+      (effects (font (size 1.27 1.27)) hide)
+    )
+    (property "Datasheet" "" (at 141.605 110.49 0)
+      (effects (font (size 1.27 1.27)) hide)
+    )
+    (pin "1")
+    (instances
+      (project "ETH2CDSO1B"
+        (path "/5e9d9a67-9011-4d17-9f7a-23dbb04d2fbf/4548d26a-48b5-4733-ae40-ebee8ab230ff"
+          (reference "#PWR0215") (unit 1)
+        )
+        (path "/5e9d9a67-9011-4d17-9f7a-23dbb04d2fbf/45cf2216-7ba0-412c-bbcb-6adbd9bfb27f"
+          (reference "#PWR0426") (unit 1)
         )
       )
@@
     )
   )
-  (symbol (lib_id "power:+12V") (at 186.055 83.82 0) (unit 1)
-    (in_bom yes) (on_board yes) (dnp no) (fields_autoplaced)
-    (property "Reference" "#PWR0233" (at 186.055 87.63 0)
-      (effects (font (size 1.27 1.27)) hide)
-    )
-    (property "Value" "+12V" (at 186.055 79.375 0)
+  (symbol (lib_id "power:+5V") (at 186.055 83.82 0) (unit 1)
+    (in_bom yes) (on_board yes) (dnp no) (fields_autoplaced)
+    (property "Reference" "#PWR0215" (at 186.055 87.63 0)
+      (effects (font (size 1.27 1.27)) hide)
+    )
+    (property "Value" "+5V" (at 186.055 79.375 0)
       (effects (font (size 1.27 1.27)))
     )
@@
       (project "ETH2CDSO1B"
         (path "/5e9d9a67-9011-4d17-9f7a-23dbb04d2fbf/4548d26a-48b5-4733-ae40-ebee8ab230ff"
-          (reference "#PWR0233") (unit 1)
-        )
-        (path "/5e9d9a67-9011-4d17-9f7a-23dbb04d2fbf/45cf2216-7ba0-412c-bbcb-6adbd9bfb27f"
+          (reference "#PWR0215") (unit 1)
+        )
+        (path "/5e9d9a67-9011-4d17-9f7a-23dbb04d2fbf/45cf2216-7ba0-412c-bbcb-6adbd9bfb27f"

Commit message: Hardware
Parts:
- removed C204, C207: 2p2, Capacitor_SMD:C_0603_1608Metric_Pad1.08x0.95mm_HandSolder, symbol Device:C
- removed C208: JR200, Capacitor_SMD:C_Trimmer_Voltronics_JR, symbol Device:C_Trim
- removed C210: 100p, Capacitor_SMD:C_0603_1608Metric_Pad1.08x0.95mm_HandSolder, symbol Device:C
- removed R207: 38k3, Resistor_SMD:R_1206_3216Metric_Pad1.30x1.75mm_HandSolder, symbol Device:R
- removed R210: 10, Resistor_SMD:R_0603_1608Metric_Pad0.98x0.95mm_HandSolder, symbol Device:R
- removed R211: 12, Resistor_SMD:R_0603_1608Metric_Pad0.98x0.95mm_HandSolder, symbol Device:R
- added C201: JR200, Capacitor_SMD:C_Trimmer_Voltronics_JR, symbol Device:C_Trim
- added C203: 22p, Capacitor_SMD:C_0603_1608Metric_Pad1.08x0.95mm_HandSolder, symbol Device:C
- added C206: 27p, Capacitor_SMD:C_0603_1608Metric_Pad1.08x0.95mm_HandSolder, symbol Device:C
- added R201: 17R8, Resistor_SMD:R_0603_1608Metric_Pad0.98x0.95mm_HandSolder, symbol Device:R
- added R203: 953k, Resistor_SMD:R_1206_3216Metric_Pad1.30x1.75mm_HandSolder, symbol Device:R
- added R204: 24k9, Resistor_SMD:R_1206_3216Metric_Pad1.30x1.75mm_HandSolder, symbol Device:R
- added R206, R209: 100, Resistor_SMD:R_0603_1608Metric_Pad0.98x0.95mm_HandSolder, symbol Device:R
- C205: value 12p -> 11p
- R202: value 100 -> 150
- R204: value 33R2 -> 4R7
- R205: value 976k -> 22k6
- R226: value 100 -> 249
- R228: value 100 -> 75
Connections:
- net LMH6552_EN_CH1 is gone; now on net LMH6552_EN_CH2: U205.7 (EN)
- net SELF_CAL_SEL_CH1 is gone; now on net SELF_CAL_SEL_CH2: K201.1
- net +12V: no longer U202.7 (V+)
- net +5V: now also U202.7 (V+)
- net GND: now also C205.2, R205.2, C201.2, C203.2
- net at K202.5, R202.2: now also C206.1, R203.1; no longer R205.1
- net at K202.4: now also R209.2
- net +5FC1 renamed +5FC2
- net -5FC1 renamed -5FC2
- new net: C201.1, C203.1, R201.1
- new net: R203.2, R204.1
- new net: R201.2, R204.2, R205.1, R206.1, R209.1
- new net: C206.2, R206.2
Other:
- moved on the sheet: C203, C206, C223, C224, FB202, R229, TP204, TP205
