File: Hardware/ETH2CDSO1B/FPGA.kicad_sch (KiCad schematic)
At the start: 18 parts, among them J601 Conn_02x01, J602 Conn_02x07_Odd_Even, U601 XC6SLX9-TQG144, U602 AT45DB161E

Commit message: Hardware
Parts:
- D601, D602: footprint (none) -> LED_SMD:LED_0603_1608Metric_Pad1.05x0.95mm_HandSolder
- R601: footprint (none) -> Resistor_SMD:R_0603_1608Metric_Pad0.98x0.95mm_HandSolder
- R602: renamed from R604; footprint (none) -> Resistor_SMD:R_0603_1608Metric_Pad0.98x0.95mm_HandSolder
- R603: renamed from R605; footprint (none) -> Resistor_SMD:R_0603_1608Metric_Pad0.98x0.95mm_HandSolder
- R604: renamed from R608; value R -> 1k; footprint (none) -> Resistor_SMD:R_0603_1608Metric_Pad0.98x0.95mm_HandSolder
- R605: renamed from R609; footprint (none) -> Resistor_SMD:R_0603_1608Metric_Pad0.98x0.95mm_HandSolder
- R606: renamed from R610; footprint (none) -> Resistor_SMD:R_0603_1608Metric_Pad0.98x0.95mm_HandSolder
- R607: renamed from R602; footprint (none) -> Resistor_SMD:R_0603_1608Metric_Pad0.98x0.95mm_HandSolder
- R608: renamed from R603; footprint (none) -> Resistor_SMD:R_0603_1608Metric_Pad0.98x0.95mm_HandSolder
- R609: renamed from R611; footprint (none) -> Resistor_SMD:R_0603_1608Metric_Pad0.98x0.95mm_HandSolder
- R610: renamed from R606; footprint (none) -> Resistor_SMD:R_0603_1608Metric_Pad0.98x0.95mm_HandSolder
- R611: renamed from R607; footprint (none) -> Resistor_SMD:R_0603_1608Metric_Pad0.98x0.95mm_HandSolder
- U601: value XC6SLX9-TQG144 -> XC6SLX9-xTQG144
- gave numbers to parts that had none: 1
