File: Hardware/ETH2CDSO1B/Voltage_Source.kicad_sch (KiCad schematic)
At the start: 6 parts, among them U301 LT1790-4.096

Commit message: Hardware
Parts:
- added C203: 10u, Capacitor_SMD:C_1206_3216Metric_Pad1.33x1.80mm_HandSolder, symbol Device:C
- added C206 (x7), C311, C312, C314, C315: 100n, Capacitor_SMD:C_0603_1608Metric_Pad1.08x0.95mm_HandSolder, symbol Device:C
- added C305, C309, C320: 1u, Capacitor_SMD:C_0603_1608Metric_Pad1.08x0.95mm_HandSolder, symbol Device:C
- added C308: 10n, Capacitor_SMD:C_0603_1608Metric_Pad1.08x0.95mm_HandSolder, symbol Device:C
- added C316, C317: 1n, Capacitor_SMD:C_0603_1608Metric_Pad1.08x0.95mm_HandSolder, symbol Device:C
- added C321, C322: 22u/16V, symbol Device:C_Polarized
- added C323: 220n, Capacitor_SMD:C_0603_1608Metric_Pad1.08x0.95mm_HandSolder, symbol Device:C
- added FB202: Z0806C251BPWZT, Inductor_SMD:L_0805_2012Metric_Pad1.15x1.40mm_HandSolder, symbol Device:FerriteBead_Small
- added Q301, Q303: BC846B, Package_TO_SOT_SMD:SOT-23, symbol Transistor_BJT:BC846
- added Q302, Q304: MMBT2907A, Package_TO_SOT_SMD:SOT-23, symbol Device:Q_PNP_BEC
- added R301, R304, R306, R311, R312: 10k, Resistor_SMD:R_0603_1608Metric_Pad0.98x0.95mm_HandSolder, symbol Device:R
- added R302, R303: 160k, Resistor_SMD:R_0603_1608Metric_Pad0.98x0.95mm_HandSolder, symbol Device:R
- added R305: 0, Resistor_SMD:R_0603_1608Metric_Pad0.98x0.95mm_HandSolder, symbol Device:R
- added R307, R309: 2k, Resistor_SMD:R_0603_1608Metric_Pad0.98x0.95mm_HandSolder, symbol Device:R
- added R308, R310: 46R4, Resistor_SMD:R_0603_1608Metric_Pad0.98x0.95mm_HandSolder, symbol Device:R
- added R313: 470, Resistor_SMD:R_0603_1608Metric_Pad0.98x0.95mm_HandSolder, symbol Device:R
- added R314, R315: 301, Resistor_SMD:R_0603_1608Metric_Pad0.98x0.95mm_HandSolder, symbol Device:R
- added R316, R317: 16k2, Resistor_SMD:R_0603_1608Metric_Pad0.98x0.95mm_HandSolder, symbol Device:R
- added R318: 75, Resistor_SMD:R_0603_1608Metric_Pad0.98x0.95mm_HandSolder, symbol Device:R
- added R319: 249, Resistor_SMD:R_0603_1608Metric_Pad0.98x0.95mm_HandSolder, symbol Device:R
- added R320: 100, symbol Device:R
- added U302: TXB0106PW, Package_SO:TSSOP-16_4.4x5mm_P0.65mm, symbol ETH2CDSO1B:TXB0106W
- added U303, U305: TLV274, Package_SO:SO-14_3.9x8.65mm_P1.27mm, symbol ETH2CDSO1B:TLV274
- added U304: DAC8568IxPW, Package_SO:TSSOP-16_4.4x5mm_P0.65mm, symbol ETH2CDSO1B:DAC8568IxPW
- added U306: TLV274, symbol ETH2CDSO1B:TLV274
Connections:
- net +5V: now also U302.15 (VCCB)
- net +5VA: now also C206.1, C206.1, C206.1, Q301.3 (C), Q303.3 (C), R304.1, U303.8 (V+), U304.3 (AVDD), U305.8 (V+), U306.8 (V+)
- net GND: now also U301.1 (GND), U301.2 (GND), C203.2, C206.2, C206.2, C206.2, C206.2, C206.2, C206.2, C206.2, C305.2, C308.2, C309.2, C311.2, C312.2, C314.2, C315.2, C320.2, C321.2, C322.2, Q302.3 (C), Q304.3 (C), R303.1, R306.1, R314.2, R315.2, U302.9 (GND), U303.5 (+), U304.14 (GND), U305.10 (+), U305.12 (+), U306.12 (+)
- net +4V: now reaches U301.6 (Vout)
- net +4V: now also C305.1, R302.1, R305.1
- new net: R306.2, U302.16 (B1), U304.1 (~{LDAC})
- new net: C315.1, U304.12 (VOUTD), U306.3 (+)
- new net: U304.13 (VOUTB), U305.5 (+)
- new net: U302.12 (B4), U304.15 (DIN)
- new net: U302.13 (B3), U304.16 (SCLK)
- new net: U302.14 (B2), U304.2 (~{SYNC})
- new net: U304.4 (VOUTA), U305.3 (+)
- new net: C314.1, U304.5 (VOUTC), U306.5 (+)
- new net: U304.6 (VOUTE), U306.10 (+)
- new net: C309.1, R305.2, U304.8 (VRFIN/VRFOUT)
- new net: R304.2, U302.11 (B5), U304.9 (~{CLR})
- new net: C311.1, C312.1, U303.12 (+), U303.3 (+), U303.8, U303.9 (-)
- new net: R311.2, R316.1, U305.13 (-)
- new net: Q301.1 (B), Q302.1 (B), R308.2
- new net: R301.2, U302.8 (OE)
- new net: U303.6 (-), U303.7
- new net: R311.1, U305.1, U305.2 (-)
- new net: C308.1, R302.2, R303.2, U303.10 (+)
- new net: C317.2, R310.1, U303.14
- new net: Q303.1 (B), Q304.1 (B), R310.2
- new net: C323.1, R319.2
- new net: C316.1, R307.1, U303.2 (-)
- new net: C316.2, R308.1, U303.1
- new net: R312.2, R317.1, U305.9 (-)
- new net: C323.2, R320.1
- new net: C317.1, R309.1, U303.13 (-)
- new net: C320.1, R318.2
- new net: R312.1, U305.6 (-), U305.7
- new net: R313.1, U306.8, U306.9 (-)
- new net: U306.13 (-), U306.14
- new net +3.3V: R301.1, U302.2 (VCCA)
- new net -5V: FB202.2
- new net -5VA: C203.1, C206.1, C206.1, C206.1, C206.1, FB202.1, U303.4 (V-), U305.4 (V-), U306.4 (V-)
- new net DAC_~{CLR}: U302.6 (A5)
- new net DAC_~{LDAC}: U302.2 (VCCA)
- new net OFFSET1_CH1: R316.2, U305.14
- new net OFFSET1_CH2: R317.2, U305.8
- new net OFFSET2_CH1: C322.1, Q303.2 (E), Q304.2 (E), R309.2, R315.1
- new net OFFSET2_CH2: C321.1, Q301.2 (E), Q302.2 (E), R307.2, R314.1
- new net OFFSET3_CH1: U306.6 (-), U306.7
- new net OFFSET3_CH2: U306.1, U306.2 (-)
- new net SELFCAL: R320.2
- new net SELF_CAL_CH1: R313.2, R318.1, R319.1
- new net SPI_CS3: U302.3 (A2)
- new net SPI_MOSI: U302.5 (A4)
- new net SPI_SCK: U302.4 (A3)
- no-connect marks 0 -> 5
Other:
- moved on the sheet: C203, C206, FB202, U301

Commit message: Hardware
Parts:
- R320: footprint (none) -> Resistor_SMD:R_0603_1608Metric_Pad0.98x0.95mm_HandSolder
- U306: footprint (none) -> Package_SO:SO-14_3.9x8.65mm_P1.27mm
Connections:
- net +5V: no longer U302.15 (VCCB)
- net +5VA: no longer C203.1, C206.1, R304.1, U301.4 (Vin), U304.3 (AVDD)
- new net +5VL: C203.1, C206.1, R304.1, U301.4 (Vin), U302.15 (VCCB), U304.3 (AVDD)
Changed lines of the file:
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@@
     )
   )
+  (symbol (lib_id "power:+5VL") (at 81.915 150.495 0) (unit 1)
+    (in_bom yes) (on_board yes) (dnp no)
+    (property "Reference" "#PWR0319" (at 81.915 154.305 0)
+      (effects (font (size 1.27 1.27)) hide)
+    )
+    (property "Value" "+5VL" (at 81.915 146.05 0)
+      (effects (font (size 1.27 1.27)))
+    )
+    (property "Footprint" "" (at 81.915 150.495 0)
+      (effects (font (size 1.27 1.27)) hide)
+    )
+    (property "Datasheet" "" (at 81.915 150.495 0)
+      (effects (font (size 1.27 1.27)) hide)
+    )
+    (pin "1")
+    (instances
+      (project "ETH2CDSO1B"
+        (path "/5e9d9a67-9011-4d17-9f7a-23dbb04d2fbf/a039f7c3-14d4-4325-8e97-2f63d3d03449"
+          (reference "#PWR0319") (unit 1)
+        )
+      )
+    )
+  )
   (symbol (lib_id "Device:C") (at 166.37 264.16 0) (unit 1)
     (in_bom yes) (on_board yes) (dnp no) (fields_autoplaced)
@@
       (effects (font (size 1.27 1.27)))
     )
-    (property "Footprint" "" (at 172.72 180.34 0)
+    (property "Footprint" "Package_SO:SO-14_3.9x8.65mm_P1.27mm" (at 172.72 180.34 0)
       (effects (font (size 1.27 1.27)) hide)
     )
@@
     )
   )
+  (symbol (lib_id "power:+5VL") (at 111.76 151.13 0) (unit 1)
+    (in_bom yes) (on_board yes) (dnp no)
+    (property "Reference" "#PWR0324" (at 111.76 154.94 0)
+      (effects (font (size 1.27 1.27)) hide)
+    )
+    (property "Value" "+5VL" (at 111.76 146.685 0)
+      (effects (font (size 1.27 1.27)))
+    )
+    (property "Footprint" "" (at 111.76 151.13 0)
+      (effects (font (size 1.27 1.27)) hide)
+    )
+    (property "Datasheet" "" (at 111.76 151.13 0)
+      (effects (font (size 1.27 1.27)) hide)
+    )
+    (pin "1")
+    (instances
+      (project "ETH2CDSO1B"
+        (path "/5e9d9a67-9011-4d17-9f7a-23dbb04d2fbf/a039f7c3-14d4-4325-8e97-2f63d3d03449"
+          (reference "#PWR0324") (unit 1)
+        )
+      )
+    )
+  )
   (symbol (lib_id "ETH2CDSO1B:TLV274") (at 189.865 163.83 0) (mirror x) (unit 3)
     (in_bom yes) (on_board yes) (dnp no)
@@
     )
   )
-  (symbol (lib_id "power:+5VA") (at 81.915 150.495 0) (unit 1)
-    (in_bom yes) (on_board yes) (dnp no) (fields_autoplaced)
-    (property "Reference" "#PWR0319" (at 81.915 154.305 0)
-      (effects (font (size 1.27 1.27)) hide)
-    )
-    (property "Value" "+5VA" (at 81.915 146.05 0)
-      (effects (font (size 1.27 1.27)))
-    )
-    (property "Footprint" "" (at 81.915 150.495 0)
-      (effects (font (size 1.27 1.27)) hide)
-    )
-    (property "Datasheet" "" (at 81.915 150.495 0)
-      (effects (font (size 1.27 1.27)) hide)
-    )
-    (pin "1")
-    (instances
-      (project "ETH2CDSO1B"
-        (path "/5e9d9a67-9011-4d17-9f7a-23dbb04d2fbf/a039f7c3-14d4-4325-8e97-2f63d3d03449"
-          (reference "#PWR0319") (unit 1)
-        )
-      )
-    )
-  )
-  (symbol (lib_id "power:+5VA") (at 40.005 39.37 0) (unit 1)
-    (in_bom yes) (on_board yes) (dnp no) (fields_autoplaced)
-    (property "Reference" "#PWR0305" (at 40.005 43.18 0)
-      (effects (font (size 1.27 1.27)) hide)
-    )
-    (property "Value" "+5VA" (at 40.005 34.925 0)
-      (effects (font (size 1.27 1.27)))
-    )
-    (property "Footprint" "" (at 40.005 39.37 0)
-      (effects (font (size 1.27 1.27)) hide)
-    )
-    (property "Datasheet" "" (at 40.005 39.37 0)
-      (effects (font (size 1.27 1.27)) hide)
-    )
-    (pin "1")
-    (instances
-      (project "ETH2CDSO1B"
-        (path "/5e9d9a67-9011-4d17-9f7a-23dbb04d2fbf/a039f7c3-14d4-4325-8e97-2f63d3d03449"
-          (reference "#PWR0305") (unit 1)
-        )
-      )
-    )
-  )
   (symbol (lib_id "Device:C") (at 208.28 232.41 0) (unit 1)
     (in_bom yes) (on_board yes) (dnp no) (fields_autoplaced)
@@
       (effects (font (size 1.27 1.27)))
     )
-    (property "Footprint" "" (at 222.885 239.903 90)
+    (property "Footprint" "Resistor_SMD:R_0603_1608Metric_Pad0.98x0.95mm_HandSolder" (at 222.885 239.903 90)
       (effects (font (size 1.27 1.27)) hide)
     )
@@
     )
   )
+  (symbol (lib_id "power:+5VL") (at 59.055 151.13 0) (unit 1)
+    (in_bom yes) (on_board yes) (dnp no)
+    (property "Reference" "#PWR0313" (at 59.055 154.94 0)
+      (effects (font (size 1.27 1.27)) hide)
+    )
+    (property "Value" "+5VL" (at 60.325 146.685 0)
+      (effects (font (size 1.27 1.27)))
+    )
+    (property "Footprint" "" (at 59.055 151.13 0)
+      (effects (font (size 1.27 1.27)) hide)
+    )
+    (property "Datasheet" "" (at 59.055 151.13 0)
+      (effects (font (size 1.27 1.27)) hide)
+    )
+    (pin "1")
+    (instances
+      (project "ETH2CDSO1B"
+        (path "/5e9d9a67-9011-4d17-9f7a-23dbb04d2fbf/a039f7c3-14d4-4325-8e97-2f63d3d03449"
+          (reference "#PWR0313") (unit 1)
+        )
+      )
+    )
+  )
   (symbol (lib_id "Device:C") (at 144.78 201.93 0) (unit 1)
     (in_bom yes) (on_board yes) (dnp no) (fields_autoplaced)
@@
     )
   )
+  (symbol (lib_id "power:+5VL") (at 40.005 39.37 0) (unit 1)
+    (in_bom yes) (on_board yes) (dnp no) (fields_autoplaced)
+    (property "Reference" "#PWR0305" (at 40.005 43.18 0)
+      (effects (font (size 1.27 1.27)) hide)
+    )
+    (property "Value" "+5VL" (at 40.005 34.29 0)
+      (effects (font (size 1.27 1.27)))
+    )
+    (property "Footprint" "" (at 40.005 39.37 0)
+      (effects (font (size 1.27 1.27)) hide)
+    )
+    (property "Datasheet" "" (at 40.005 39.37 0)
+      (effects (font (size 1.27 1.27)) hide)
+    )
+    (pin "1")
+    (instances
+      (project "ETH2CDSO1B"
+        (path "/5e9d9a67-9011-4d17-9f7a-23dbb04d2fbf/a039f7c3-14d4-4325-8e97-2f63d3d03449"
+          (reference "#PWR0305") (unit 1)
+        )
+      )
+    )
+  )
   (symbol (lib_id "ETH2CDSO1B:TLV274") (at 138.43 84.455 0) (mirror x) (unit 4)
     (in_bom yes) (on_board yes) (dnp no)
@@
       (effects (font (size 1.27 1.27)))
     )
-    (property "Footprint" "" (at 172.72 199.39 0)
+    (property "Footprint" "Package_SO:SO-14_3.9x8.65mm_P1.27mm" (at 172.72 199.39 0)
       (effects (font (size 1.27 1.27)) hide)
     )
@@
       (effects (font (size 1.27 1.27)))
     )
-    (property "Footprint" "" (at 172.72 219.71 0)
+    (property "Footprint" "Package_SO:SO-14_3.9x8.65mm_P1.27mm" (at 172.72 219.71 0)
       (effects (font (size 1.27 1.27)) hide)
     )
@@
     )
   )
-  (symbol (lib_id "power:+5VA") (at 111.76 151.13 0) (unit 1)
-    (in_bom yes) (on_board yes) (dnp no) (fields_autoplaced)
-    (property "Reference" "#PWR0324" (at 111.76 154.94 0)
-      (effects (font (size 1.27 1.27)) hide)
-    )
-    (property "Value" "+5VA" (at 111.76 146.685 0)
-      (effects (font (size 1.27 1.27)))
-    )
-    (property "Footprint" "" (at 111.76 151.13 0)
-      (effects (font (size 1.27 1.27)) hide)
-    )
-    (property "Datasheet" "" (at 111.76 151.13 0)
-      (effects (font (size 1.27 1.27)) hide)
-    )
-    (pin "1")
-    (instances
-      (project "ETH2CDSO1B"
-        (path "/5e9d9a67-9011-4d17-9f7a-23dbb04d2fbf/a039f7c3-14d4-4325-8e97-2f63d3d03449"
-          (reference "#PWR0324") (unit 1)
-        )
-      )
-    )
-  )
   (symbol (lib_id "power:-5VA") (at 244.475 271.78 180) (unit 1)
     (in_bom yes) (on_board yes) (dnp no) (fields_autoplaced)
@@
       (effects (font (size 1.27 1.27)) (justify left))
     )
-    (property "Footprint" "" (at 243.205 264.16 0)
+    (property "Footprint" "Package_SO:SO-14_3.9x8.65mm_P1.27mm" (at 243.205 264.16 0)
       (effects (font (size 1.27 1.27)) hide)
     )
@@
   )
   (symbol (lib_id "power:+3.3V") (at 53.975 151.13 0) (unit 1)
-    (in_bom yes) (on_board yes) (dnp no) (fields_autoplaced)
+    (in_bom yes) (on_board yes) (dnp no)
     (property "Reference" "#PWR0310" (at 53.975 154.94 0)
       (effects (font (size 1.27 1.27)) hide)
     )
-    (property "Value" "+3.3V" (at 53.975 146.685 0)
+    (property "Value" "+3.3V" (at 52.705 146.685 0)
       (effects (font (size 1.27 1.27)))
     )
@@
     )
   )
-  (symbol (lib_id "power:+5V") (at 59.055 151.13 0) (unit 1)
-    (in_bom yes) (on_board yes) (dnp no) (fields_autoplaced)
-    (property "Reference" "#PWR0215" (at 59.055 154.94 0)
-      (effects (font (size 1.27 1.27)) hide)
-    )
-    (property "Value" "+5V" (at 59.055 146.685 0)
-      (effects (font (size 1.27 1.27)))
-    )
-    (property "Footprint" "" (at 59.055 151.13 0)
-      (effects (font (size 1.27 1.27)) hide)
-    )
-    (property "Datasheet" "" (at 59.055 151.13 0)
-      (effects (font (size 1.27 1.27)) hide)
-    )
-    (pin "1")
-    (instances
-      (project "ETH2CDSO1B"
-        (path "/5e9d9a67-9011-4d17-9f7a-23dbb04d2fbf/4548d26a-48b5-4733-ae40-ebee8ab230ff"
-          (reference "#PWR0215") (unit 1)
-        )
-        (path "/5e9d9a67-9011-4d17-9f7a-23dbb04d2fbf/a039f7c3-14d4-4325-8e97-2f63d3d03449"
-          (reference "#PWR0313") (unit 1)
-        )
-      )
-    )
-  )
   (symbol (lib_id "power:-5VA") (at 114.3 257.81 0) (unit 1)
     (in_bom yes) (on_board yes) (dnp no)
@@
       (effects (font (size 1.27 1.27)))
     )
-    (property "Footprint" "" (at 281.94 257.81 0)
+    (property "Footprint" "Package_SO:SO-14_3.9x8.65mm_P1.27mm" (at 281.94 257.81 0)
       (effects (font (size 1.27 1.27)) hide)
     )
